File: pcb/bolide-65-pcb.kicad_pcb (KiCad board)
At the start: 2 copper layers, 307 x 101 mm, 270 parts, among them SW1 Backtick, SW10 9, SW11 0, SW12 Minus, SW13 Equals, SW14 Backspace, SW15 Tab, SW16 Q, SW17 W, SW18 E, SW19 R, SW2 1, SW20 T, SW21 Y, SW22 U, SW23 I, SW24 O, SW25 P, SW26 LBracket, SW27 RBracket, SW28 Backslash, SW29 CapsLock, SW3 2, SW30 A, SW31 S, SW32 D, SW33 F, SW34 G, SW35 H, SW36 J, SW37 K, SW38 L, SW39 Semicolon, SW4 3, SW40 Quote, SW41 Enter, SW42 PgUp, SW43 LShift, SW44 Z, SW45 X, SW46 C, SW47 V, SW48 B, SW49 N, SW5 4, SW50 M, SW51 Comma, SW52 Period, SW53 Slash, SW54 RShift, SW55 Up, SW56 PgDown, SW57 LCtrl, SW58 Menu, SW59 LAlt, SW6 5, SW60 Space, SW61 RAlt, SW62 Fn, SW63 Blank, SW64 Left, SW65 Down, SW66 Right, SW7 6, SW8 7, SW9 8, U1 RP2040-ZERO, U2 74AHCT1G125

Commit message: update pcb files w/ improved silkscreen
Parts:
- added G***: LOGO, LOGO, F.Cu at (365.1, 50.4)
- added G***: LOGO, LOGO, F.Cu at (364.9, 42.9)
Routing:
- net Net-(LED60-DOUT): track 110.8 -> 106.0 mm
- net +5V: track 2181.4 -> 2184.3 mm
- net COL1: track 767.7 -> 765.9 mm
Other:
- board text added: "Bolide65"
- board text added: "RP2040 Zero"
- board text added: "v1.0 // 11.10.2026"
- board text added: "© Reuben O"
